Commit message: Rviz 3D Puzzlebot working (Need to change joint type later)

File: localisation/urdf/puzzlebot_jetson_ed_urdf.urdf (robot description, URDF)
Before this commit: robot Puzzlebot Jetson-Lidar Ed., 2 links, 1 joints
Links:
- added link wl_link; collision mesh filename=package://localisation/models/MCR2_1000_1_1_Wheel_Coupler_2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; visual mesh filename=package://localisation/models/MCR2_1000_1_1_Wheel_Coupler_2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
- added link wr_link, mass 0.03; collision mesh filename=package://localisation/models/MCR2_1000_1_1_Wheel_Coupler_2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; visual mesh filename=package://localisation/models/MCR2_1000_1_1_Wheel_Coupler_2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
Joints:
- added joint leftWheel: type fixed, parent chassis, child wl_link, origin xyz=0.05 0.0955 0
- added joint rightWheel: type fixed, parent chassis, child wr_link, origin xyz=0.05 -0.0955 0

Commit message: Part 2 Done :) Rviz and Joint State Pub and TFs

File: localisation/urdf/puzzlebot_jetson_ed_urdf.urdf (robot description, URDF)
Before this commit: robot Puzzlebot Jetson-Lidar Ed., 4 links, 3 joints
Links:
- link wl_link: mass None -> 0.03
Joints:
- joint leftWheel: axis (none) -> 0 1 0; type fixed -> continuous
- joint rightWheel: axis (none) -> 0 1 0; type fixed -> continuous
